Commit message: No funciona correctamente

File: robots/robot_B.urdf.xacro (robot description, xacro)
@@ -2,13 +2,11 @@
 <!-- created with Phobos 1.0.1 "Capricious Choutengan" -->
   <robot name="robot" xmlns:xacro="http://wiki.ros.org/xacro">
+    <xacro:include filename="$(find robot_description)/urdf/control/ros2_control.urdf.xacro"/>
+    <xacro:arg name="config_controllers" default="$(find robot_description)/config/rover_controller.yaml/"/>
+    <xacro:arg name="update_rate" default="100"/>
+    <xacro:ros2_control/>
     <xacro:include filename="$(find robot_description)/urdf/sensors/sensors.urdf.xacro"/>
     <xacro:arg name="prefix" default=""/>
     <xacro:arg name="my_robot" default=""/>
-    <!-- <xacro:include filename="$(find robot_description)/urdf/wheels/wheels.urdf.xacro"/>
-    <xacro:arg name="prefix" default=""/> -->
-    <xacro:include filename="$(find robot_description)/urdf/control/ros2_control.urdf.xacro"/>
-    <xacro:arg name="config_controllers" default="$(find robot_description)/config/wheels_controller.yaml/"/>
-    <xacro:arg name="update_rate" default="100"/>
-    <xacro:ros2_control/>
     <link name="base_footprint">
       <origin xyz="0 0 0" rpy="0 0 0"/>
@@ -216,5 +214,5 @@
       <child link="back_left_wheel"/>
       <axis xyz="0 0 1.0"/>
-      <limit effort="0" velocity="0"/>
+      <limit effort="5000" velocity="100"/>
     </joint>
     <joint name="front_left_wheel_joint" type="continuous">
@@ -223,5 +221,5 @@
       <child link="front_left_wheel"/>
       <axis xyz="0 0 1.0"/>
-      <limit effort="0" velocity="0"/>
+      <limit effort="5000" velocity="100"/>
     </joint>
     <joint name="back_right_wheel_joint" type="continuous">
@@ -230,5 +228,5 @@
       <child link="back_right_wheel"/>
       <axis xyz="0 0 1.0"/>
-      <limit effort="0" velocity="0"/>
+      <limit effort="5000" velocity="100"/>
     </joint>
     <joint name="front_right_wheel_joint" type="continuous">
@@ -237,5 +235,5 @@
       <child link="front_right_wheel"/>
       <axis xyz="0 0 1.0"/>
-      <limit effort="0" velocity="0"/>
+      <limit effort="5000" velocity="100"/>
     </joint>
     <transmission name="$back_left_wheel_joint_trans">

Commit message: Robot se configura y spawnea correctamente

File: robots/robot_B.urdf.xacro (robot description, xacro)
@@ -3,5 +3,5 @@
   <robot name="robot" xmlns:xacro="http://wiki.ros.org/xacro">
     <xacro:include filename="$(find robot_description)/urdf/control/ros2_control.urdf.xacro"/>
-    <xacro:arg name="config_controllers" default="$(find robot_description)/config/rover_controller.yaml/"/>
+    <xacro:arg name="config_controllers" default="$(find robot_description)/config/wheels_controller.yaml"/>
     <xacro:arg name="update_rate" default="100"/>
     <xacro:ros2_control/>
@@ -237,53 +237,53 @@
       <limit effort="5000" velocity="100"/>
     </joint>
-    <transmission name="$back_left_wheel_joint_trans">
+    <transmission name="back_left_wheel_joint_trans">
       <type>transmission_interface/SimpleTransmission</type>
-      <joint name="$back_left_wheel_joint">
+      <joint name="back_left_wheel_joint">
         <hardwareInterface>hardware_interface/VelocityJointInterface</hardwareInterface>
       </joint>
-      <actuator name="$back_left_wheel_joint_motor">
+      <actuator name="back_left_wheel_joint_motor">
         <mechanicalReduction>1</mechanicalReduction>
       </actuator>
     </transmission>
-    <gazebo reference="$back_left_wheel">
+    <gazebo reference="back_left_wheel">
       <mu1>5</mu1>
       <mu2>5</mu2>
     </gazebo>
-    <transmission name="$front_left_wheel_joint_trans">
+    <transmission name="front_left_wheel_joint_trans">
       <type>transmission_interface/SimpleTransmission</type>
-      <joint name="$front_left_wheel_joint">
+      <joint name="front_left_wheel_joint">
         <hardwareInterface>hardware_interface/VelocityJointInterface</hardwareInterface>
       </joint>
-      <actuator name="$front_left_wheel_joint_motor">
+      <actuator name="front_left_wheel_joint_motor">
         <mechanicalReduction>1</mechanicalReduction>
       </actuator>
     </transmission>
-    <gazebo reference="$front_left_wheel">
+    <gazebo reference="front_left_wheel">
       <mu1>5</mu1>
       <mu2>5</mu2>
     </gazebo>
-    <transmission name="$back_right_wheel_joint_trans">
+    <transmission name="back_right_wheel_joint_trans">
       <type>transmission_interface/SimpleTransmission</type>
-      <joint name="$back_right_wheel_joint">
+      <joint name="back_right_wheel_joint">
         <hardwareInterface>hardware_interface/VelocityJointInterface</hardwareInterface>
       </joint>
-      <actuator name="$back_right_wheel_joint_motor">
+      <actuator name="back_right_wheel_joint_motor">
         <mechanicalReduction>1</mechanicalReduction>
       </actuator>
     </transmission>
-    <gazebo reference="$back_right_wheel">
+    <gazebo reference="back_right_wheel">
       <mu1>5</mu1>
       <mu2>5</mu2>
     </gazebo>
-    <transmission name="$front_right_wheel_joint_trans">
+    <transmission name="front_right_wheel_joint_trans">
       <type>transmission_interface/SimpleTransmission</type>
-      <joint name="$front_right_wheel_joint">
+      <joint name="front_right_wheel_joint">
         <hardwareInterface>hardware_interface/VelocityJointInterface</hardwareInterface>
       </joint>
-      <actuator name="$front_right_wheel_joint_motor">
+      <actuator name="front_right_wheel_joint_motor">
         <mechanicalReduction>1</mechanicalReduction>
       </actuator>
     </transmission>
-    <gazebo reference="$front_right_wheel">
+    <gazebo reference="front_right_wheel">
       <mu1>5</mu1>
       <mu2>5</mu2>
