Commit message: Terminado

File: robots/robot_A.urdf.xacro (robot description, xacro)
@@ -416,4 +416,3 @@
       <origin xyz="0.0 0.0 0.0" rpy="0 0 0"/>
     </xacro:sensor_imu>
-    <!-- </xacro:macro> -->
 </robot>

File: robots/robot_B.urdf.xacro (robot description, xacro)
@@ -185,5 +185,5 @@
     </link>
     <joint name="base_joint" type="fixed">
-      <origin xyz="0 0 0.5" rpy="0 0 0"/>
+      <origin xyz="0 0 0.8" rpy="0 0 0"/>
       <parent link="base_footprint"/>
       <child link="base_link"/>
@@ -223,6 +223,7 @@
       <limit effort="5000" velocity="100"/>
     </joint>
+    <!-- RPY modified -->
     <joint name="back_right_wheel_joint" type="continuous">
-      <origin xyz="-1.0 -1.05 -0.5" rpy="-1.5708 0 0"/>
+      <origin xyz="-1.0 -1.05 -0.5" rpy="1.5708 0 0"/>
       <parent link="base_link"/>
       <child link="back_right_wheel"/>
@@ -231,5 +232,5 @@
     </joint>
     <joint name="front_right_wheel_joint" type="continuous">
-      <origin xyz="1.0 -1.05 -0.5" rpy="-1.5708 0 0"/>
+      <origin xyz="1.0 -1.05 -0.5" rpy="1.5708 0 0"/>
       <parent link="base_link"/>
       <child link="front_right_wheel"/>
@@ -237,4 +238,5 @@
       <limit effort="5000" velocity="100"/>
     </joint>
+    <!--  -->
     <transmission name="back_left_wheel_joint_trans">
       <type>transmission_interface/SimpleTransmission</type>

File: urdf/control/ros2_control.urdf.xacro (robot description, xacro)
@@ -7,5 +7,5 @@
         </plugin>
       </gazebo>
-      <ros2_control name="rover_interface" type="system">
+      <ros2_control name="robot_interface" type="system">
         <hardware>
           <plugin>gazebo_ros2_control/GazeboSystem</plugin>

Commit message: Pulidos cambios finales

File: robots/robot_A.urdf.xacro (robot description, xacro)
@@ -410,8 +410,11 @@
       <color rgba="0.64 0.64 0.64 1.0"/>
     </material>
-    <xacro:sensor_camera node_name="arm_camera" node_namespace="$(arg my_robot)" frame_prefix="$(arg prefix)arm_camera_" parent="$(arg prefix)base_arm" >
-      <origin xyz="0.0 0.0 -0.01" rpy="0 3.141592 0"/>
+    <xacro:sensor_camera node_name="base_camera" node_namespace="$(arg my_robot)" frame_prefix="$(arg prefix)base_" parent="$(arg prefix)base_link" >
+      <origin xyz="1.5 0.0 -0.01" rpy="0 0 0"/>
     </xacro:sensor_camera>
-    <xacro:sensor_imu ns="$(arg my_robot)" prefix="$(arg prefix)imu_" parent="$(arg prefix)base_link">
+    <xacro:sensor_camera node_name="arm_camera" node_namespace="$(arg my_robot)" frame_prefix="$(arg prefix)arm_" parent="$(arg prefix)end_effector" >
+      <origin xyz="0.2 0.0 -0.01" rpy="0 0 0"/>
+    </xacro:sensor_camera>
+    <xacro:sensor_imu ns="$(arg my_robot)" prefix="$(arg prefix)imu" parent="$(arg prefix)base_link">
       <origin xyz="0.0 0.0 0.0" rpy="0 0 0"/>
     </xacro:sensor_imu>

File: robots/robot_B.urdf.xacro (robot description, xacro)
@@ -225,5 +225,5 @@
     <!-- RPY modified -->
     <joint name="back_right_wheel_joint" type="continuous">
-      <origin xyz="-1.0 -1.05 -0.5" rpy="1.5708 0 0"/>
+      <origin xyz="-1.0 -1.05 -0.5" rpy="-1.5708 0 0"/>
       <parent link="base_link"/>
       <child link="back_right_wheel"/>
@@ -232,5 +232,5 @@
     </joint>
     <joint name="front_right_wheel_joint" type="continuous">
-      <origin xyz="1.0 -1.05 -0.5" rpy="1.5708 0 0"/>
+      <origin xyz="1.0 -1.05 -0.5" rpy="-1.5708 0 0"/>
       <parent link="base_link"/>
       <child link="front_right_wheel"/>
@@ -294,21 +294,9 @@
       <color rgba="0.64 0.64 0.64 1.0"/>
     </material>
-    <xacro:sensor_camera node_name="arm_camera" node_namespace="$(arg my_robot)" frame_prefix="$(arg prefix)arm_camera_" parent="$(arg prefix)base_link" >
-      <origin xyz="0.0 0.0 -0.01" rpy="0 3.141592 0"/>
+    <xacro:sensor_camera node_name="base_camera" node_namespace="$(arg my_robot)" frame_prefix="$(arg prefix)base_" parent="$(arg prefix)base_link" >
+      <origin xyz="1.5 0.0 -0.01" rpy="0 0 0"/>
     </xacro:sensor_camera>
-    <xacro:sensor_imu ns="$(arg my_robot)" prefix="$(arg prefix)imu_" parent="$(arg prefix)base_link">
+    <xacro:sensor_imu ns="$(arg my_robot)" prefix="$(arg prefix)imu" parent="$(arg prefix)base_link">
       <origin xyz="0.0 0.0 0.0" rpy="0 0 0"/>
     </xacro:sensor_imu>
-    <!-- <xacro:robot_wheel prefix="left_b" parent="base_link" >
-      <origin xyz="-1.0 1.05 -0.5" rpy="-1.5708 0 0"/>
-    </xacro:robot_wheel>
-    <xacro:robot_wheel prefix="left_f" parent="base_link" >
-      <origin xyz="1.0 1.05 -0.5" rpy="-1.5708 0 0"/>
-    </xacro:robot_wheel>
-    <xacro:robot_wheel prefix="right_b" parent="base_link" >
-      <origin xyz="-1.0 -1.05 -0.5" rpy="-1.5708 0 0"/>
-    </xacro:robot_wheel>
-    <xacro:robot_wheel prefix="right_f" parent="base_link" >
-      <origin xyz="1.0 -1.05 -0.5" rpy="-1.5708 0 0"/>
-    </xacro:robot_wheel> -->
 </robot>
